Commit message: Update caster wheel dimensions and friction parameters for improved stability in simulation

File: src/campus_robot/urdf/wheels.xacro (robot description, xacro)
@@ -86,5 +86,5 @@
         <visual>
             <geometry>
-                <sphere radius="0.04"/>   <!-- bigger radius — more stable -->
+                <sphere radius="0.05"/>   <!-- bigger radius — more stable -->
             </geometry>
             <material name="grey"/>
@@ -92,5 +92,5 @@
         <collision>
             <geometry>
-                <sphere radius="0.04"/>
+                <sphere radius="0.05"/>
             </geometry>
         </collision>
@@ -110,5 +110,5 @@
         <parent link="base_link"/>
         <child link="caster_wheel_left"/>
-        <origin xyz="-0.17 0.10 0.05"/>  <!-- rear, spread left -->
+        <origin xyz="-0.17 0.10 0.06"/>  <!-- rear, spread left -->
     </joint>
     <!-- ============================= -->
@@ -118,5 +118,5 @@
         <visual>
             <geometry>
-                <sphere radius="0.04"/>
+                <sphere radius="0.05"/>
             </geometry>
             <material name="grey"/>
@@ -124,5 +124,5 @@
         <collision>
             <geometry>
-                <sphere radius="0.04"/>
+                <sphere radius="0.05"/>
             </geometry>
         </collision>
@@ -142,5 +142,5 @@
         <parent link="base_link"/>
         <child link="caster_wheel_right"/>
-        <origin xyz="-0.17 -0.10 0.05"/>  <!-- rear, spread right -->
+        <origin xyz="-0.17 -0.10 0.06"/>  <!-- rear, spread right -->
     </joint>
 </robot>
