Commit message: Revise LiDAR section in sensors.xacro: update geometry, add inertial properties, and adjust joint parameters

File: src/campus_robot/urdf/sensors.xacro (robot description, xacro)
@@ -35,29 +35,58 @@
         <origin xyz="0.14 0 0.19"/>
     </joint>
-    <!-- ===================================== -->
-    <!-- LiDAR                                 -->
-    <!-- ===================================== -->
-    <link name="lidar_link">
-        <visual>
-            <geometry>
-                <cylinder radius="0.045"
-                          length="0.05"/>
-            </geometry>
-            <material name="dark_grey"/>
-        </visual>
-        <collision>
-            <geometry>
-                <cylinder radius="0.045"
-                          length="0.05"/>
-            </geometry>
-        </collision>
-    </link>
-    <joint
-        name="lidar_joint"
-        type="fixed">
-        <parent link="sensor_tower"/>
-        <child link="lidar_link"/>
-        <origin xyz="0 0 0.095"/>
-    </joint>
+<!-- ═══════════════════════════════════════════════════════
+     sensors.xacro  —  LiDAR section (revised)
+     Assumes sensor_tower top is at z ≈ 0.30 m above base_link
+     ═══════════════════════════════════════════════════════ -->
+  <!-- ── LiDAR mount ring (purely visual, tiny) ── -->
+  <link name="lidar_base_link">
+    <visual>
+      <geometry>
+        <cylinder radius="0.045" length="0.02"/>
+      </geometry>
+      <material name="dark_grey"/>
+    </visual>
+    <!-- No <collision> here — keeps the scan rays unblocked -->
+    <inertial>
+      <mass value="0.05"/>
+      <inertia ixx="0.0001" ixy="0" ixz="0"
+               iyy="0.0001" iyz="0"
+               izz="0.0001"/>
+    </inertial>
+  </link>
+  <!-- Mount ring sits on TOP of the sensor tower -->
+  <joint name="lidar_base_joint" type="fixed">
+    <parent link="sensor_tower"/>
+    <child  link="lidar_base_link"/>
+    <origin xyz="0.0 0.0 0.08" rpy="0 0 0"/>
+  </joint>
+  <!-- ── LiDAR sensor link — the actual scan frame ── -->
+  <link name="lidar_link">
+    <visual>
+      <geometry>
+        <!-- Thin disc — represents the rotating head -->
+        <cylinder radius="0.04" length="0.04"/>
+      </geometry>
+      <material name="black"/>
+    </visual>
+    <!-- CRITICAL: collision is a near-zero box so rays are not blocked -->
+    <collision>
+      <geometry>
+        <box size="0.001 0.001 0.001"/>
+      </geometry>
+    </collision>
+    <inertial>
+      <mass value="0.1"/>
+      <inertia ixx="0.0001" ixy="0" ixz="0"
+               iyy="0.0001" iyz="0"
+               izz="0.0001"/>
+    </inertial>
+  </link>
+  <!-- lidar_link sits 0.03 m above the mount ring -->
+  <joint name="lidar_joint" type="fixed">
+    <parent link="lidar_base_link"/>
+    <child  link="lidar_link"/>
+    <origin xyz="0.0 0.0 0.03" rpy="0 0 0"/>
+  </joint>
     <!-- ===================================== -->
     <!-- Camera Mount                          -->
@@ -81,5 +110,5 @@
         <parent link="sensor_tower"/>
         <child link="camera_mount"/>
-        <origin xyz="0.05 0 0.02"/>
+        <origin xyz="0.05 0 0.04"/>
     </joint>
     <!-- ===================================== -->

Commit message: Update launch and URDF files: enhance robot description handling and improve LiDAR component definitions

File: src/campus_robot/urdf/sensors.xacro (robot description, xacro)
@@ -28,4 +28,14 @@
         </inertial>
     </link>
+    <!-- ─────────────────────────────────────────────────────────────
+         sensor_tower_joint: z = 0.19 m from base_link
+         Tower half-height   = 0.07 m  →  tower top = 0.19 + 0.07 = 0.26 m
+         Parcel box top      = 0.12 + 0.18 + 0.06   = 0.36 m  (the obstacle)
+         LiDAR must clear    ≥ 0.37 m from base_link
+         From tower centre:  0.37 - 0.19 = 0.18 m needed total offset
+         Split: lidar_base_joint z = 0.15 m  (clears tower top: 0.07 + margin)
+                lidar_joint      z = 0.03 m
+                Total from base_link: 0.19 + 0.15 + 0.03 = 0.37 m ✓
+    ───────────────────────────────────────────────────────────────── -->
     <joint
         name="sensor_tower_joint"
@@ -35,60 +45,67 @@
         <origin xyz="0.14 0 0.19"/>
     </joint>
-<!-- ═══════════════════════════════════════════════════════
-     sensors.xacro  —  LiDAR section (revised)
-     Assumes sensor_tower top is at z ≈ 0.30 m above base_link
-     ═══════════════════════════════════════════════════════ -->
-  <!-- ── LiDAR mount ring (purely visual, tiny) ── -->
-  <link name="lidar_base_link">
-    <visual>
-      <geometry>
-        <cylinder radius="0.045" length="0.02"/>
-      </geometry>
-      <material name="dark_grey"/>
-    </visual>
-    <!-- No <collision> here — keeps the scan rays unblocked -->
-    <inertial>
-      <mass value="0.05"/>
-      <inertia ixx="0.0001" ixy="0" ixz="0"
-               iyy="0.0001" iyz="0"
-               izz="0.0001"/>
-    </inertial>
-  </link>
-  <!-- Mount ring sits on TOP of the sensor tower -->
-  <joint name="lidar_base_joint" type="fixed">
-    <parent link="sensor_tower"/>
-    <child  link="lidar_base_link"/>
-    <origin xyz="0.0 0.0 0.08" rpy="0 0 0"/>
-  </joint>
-  <!-- ── LiDAR sensor link — the actual scan frame ── -->
-  <link name="lidar_link">
-    <visual>
-      <geometry>
-        <!-- Thin disc — represents the rotating head -->
-        <cylinder radius="0.04" length="0.04"/>
-      </geometry>
-      <material name="black"/>
-    </visual>
-    <!-- CRITICAL: collision is a near-zero box so rays are not blocked -->
-    <collision>
-      <geometry>
-        <box size="0.001 0.001 0.001"/>
-      </geometry>
-    </collision>
-    <inertial>
-      <mass value="0.1"/>
-      <inertia ixx="0.0001" ixy="0" ixz="0"
-               iyy="0.0001" iyz="0"
-               izz="0.0001"/>
-    </inertial>
-  </link>
-  <!-- lidar_link sits 0.03 m above the mount ring -->
-  <joint name="lidar_joint" type="fixed">
-    <parent link="lidar_base_link"/>
-    <child  link="lidar_link"/>
-    <origin xyz="0.0 0.0 0.03" rpy="0 0 0"/>
-  </joint>
+    <!-- ================================ -->
+    <!-- LiDAR Mount Ring                 -->
+    <!-- (no collision — visual only)     -->
+    <!-- ================================ -->
+    <link name="lidar_base_link">
+        <visual>
+            <geometry>
+                <cylinder radius="0.045" length="0.02"/>
+            </geometry>
+            <material name="dark_grey"/>
+        </visual>
+        <!-- NO collision block — mount ring must not block laser rays -->
+        <inertial>
+            <mass value="0.05"/>
+            <inertia ixx="0.0001" ixy="0" ixz="0"
+                     iyy="0.0001" iyz="0"
+                     izz="0.0001"/>
+        </inertial>
+    </link>
+    <!-- z=0.15 from tower centre → puts mount ring at 0.19+0.15 = 0.34 m -->
+    <!-- That is already above parcel box top (0.36 m)... wait:             -->
+    <!-- 0.34 m mount + 0.03 m lidar_joint = 0.37 m for lidar_link ✓       -->
+    <joint name="lidar_base_joint" type="fixed">
+        <parent link="sensor_tower"/>
+        <child  link="lidar_base_link"/>
+        <origin xyz="0.0 0.0 0.15" rpy="0 0 0"/>
+    </joint>
+    <!-- ================================ -->
+    <!-- LiDAR Sensor Link                -->
+    <!-- (scan frame — tiny collision)    -->
+    <!-- ================================ -->
+    <link name="lidar_link">
+        <visual>
+            <geometry>
+                <!-- Thin rotating disc — purely cosmetic -->
+                <cylinder radius="0.04" length="0.04"/>
+            </geometry>
+            <material name="black"/>
+        </visual>
+        <!-- Near-zero collision so rays never hit the lidar body itself -->
+        <collision>
+            <geometry>
+                <box size="0.001 0.001 0.001"/>
+            </geometry>
+        </collision>
+        <inertial>
+            <mass value="0.1"/>
+            <inertia ixx="0.0001" ixy="0" ixz="0"
+                     iyy="0.0001" iyz="0"
+                     izz="0.0001"/>
+        </inertial>
+    </link>
+    <!-- lidar_link = 0.03 m above mount ring                              -->
+    <!-- Final height from base_link: 0.19 + 0.15 + 0.03 = 0.37 m        -->
+    <!-- Parcel box top = 0.36 m  →  LiDAR clears by 1 cm ✓               -->
+    <joint name="lidar_joint" type="fixed">
+        <parent link="lidar_base_link"/>
+        <child  link="lidar_link"/>
+        <origin xyz="0.0 0.0 0.03" rpy="0 0 0"/>
+    </joint>
     <!-- ===================================== -->
     <!-- Camera Mount                          -->
+    <!-- (no collision — must not block scans) -->
     <!-- ===================================== -->
     <link name="camera_mount">
@@ -99,9 +116,5 @@
             <material name="dark_grey"/>
         </visual>
-        <collision>
-            <geometry>
-                <box size="0.03 0.03 0.05"/>
-            </geometry>
-        </collision>
+        <!-- NO collision block — camera mount must not block LiDAR rays -->
     </link>
     <joint
@@ -114,4 +127,5 @@
     <!-- ===================================== -->
     <!-- RGB Camera                            -->
+    <!-- (no collision — must not block scans) -->
     <!-- ===================================== -->
     <link name="camera_link">
@@ -122,9 +136,5 @@
             <material name="black"/>
         </visual>
-        <collision>
-            <geometry>
-                <box size="0.05 0.04 0.04"/>
-            </geometry>
-        </collision>
+        <!-- NO collision block — camera body must not block LiDAR rays -->
     </link>
     <joint

Commit message: Update LiDAR and camera joint parameters: adjust mount height and origin positions

File: src/campus_robot/urdf/sensors.xacro (robot description, xacro)
@@ -64,5 +64,5 @@
         </inertial>
     </link>
-    <!-- z=0.15 from tower centre → puts mount ring at 0.19+0.15 = 0.34 m -->
+    <!-- z=0.20 from tower centre → puts mount ring at 0.19+0.20 = 0.39 m -->
     <!-- That is already above parcel box top (0.36 m)... wait:             -->
     <!-- 0.34 m mount + 0.03 m lidar_joint = 0.37 m for lidar_link ✓       -->
@@ -70,5 +70,5 @@
         <parent link="sensor_tower"/>
         <child  link="lidar_base_link"/>
-        <origin xyz="0.0 0.0 0.15" rpy="0 0 0"/>
+        <origin xyz="0.0 0.0 0.20" rpy="0 0 0"/>
     </joint>
     <!-- ================================ -->
@@ -123,5 +123,5 @@
         <parent link="sensor_tower"/>
         <child link="camera_mount"/>
-        <origin xyz="0.05 0 0.04"/>
+        <origin xyz="0.04 0 -0.04"/>
     </joint>
     <!-- ===================================== -->

Commit message: Enhance URDF by adding visual, collision, and inertial properties for lidar posts to improve simulation fidelity

File: src/campus_robot/urdf/sensors.xacro (robot description, xacro)
@@ -176,14 +176,32 @@
         <origin xyz="0.20 0.07 0.265"/>
     </joint>
-    <link name="lidar_post_fr">  ... same geometry ...  </link>
+     <link name="lidar_post_fr">
+        <visual><geometry><box size="0.015 0.015 0.25"/></geometry><material name="black"/></visual>
+        <collision><geometry><box size="0.015 0.015 0.25"/></geometry></collision>
+        <inertial><mass value="0.15"/><origin xyz="0 0 0"/>
+            <inertia ixx="0.001" ixy="0" ixz="0" iyy="0.001" iyz="0" izz="0.00005"/></inertial>
+    </link>
     <joint name="lidar_post_fr_joint" type="fixed">
+        <parent link="base_link"/><child link="lidar_post_fr"/>
         <origin xyz="0.20 -0.07 0.265"/>
     </joint>
-    <link name="lidar_post_rl">  ... same geometry ...  </link>
+    <link name="lidar_post_rl">
+        <visual><geometry><box size="0.015 0.015 0.25"/></geometry><material name="black"/></visual>
+        <collision><geometry><box size="0.015 0.015 0.25"/></geometry></collision>
+        <inertial><mass value="0.15"/><origin xyz="0 0 0"/>
+            <inertia ixx="0.001" ixy="0" ixz="0" iyy="0.001" iyz="0" izz="0.00005"/></inertial>
+    </link>
     <joint name="lidar_post_rl_joint" type="fixed">
+        <parent link="base_link"/><child link="lidar_post_rl"/>
         <origin xyz="0.08 0.07 0.265"/>
     </joint>
-    <link name="lidar_post_rr">  ... same geometry ...  </link>
+    <link name="lidar_post_rr">
+        <visual><geometry><box size="0.015 0.015 0.25"/></geometry><material name="black"/></visual>
+        <collision><geometry><box size="0.015 0.015 0.25"/></geometry></collision>
+        <inertial><mass value="0.15"/><origin xyz="0 0 0"/>
+            <inertia ixx="0.001" ixy="0" ixz="0" iyy="0.001" iyz="0" izz="0.00005"/></inertial>
+    </link>
     <joint name="lidar_post_rr_joint" type="fixed">
+        <parent link="base_link"/><child link="lidar_post_rr"/>
         <origin xyz="0.08 -0.07 0.265"/>
     </joint>

Commit message: Update lidar post dimensions and joint origins in URDF for improved simulation accuracy

File: src/campus_robot/urdf/sensors.xacro (robot description, xacro)
@@ -167,6 +167,6 @@
     <!-- bottom z=0.14 (2mm above chassis top), top z=0.39 (below LiDAR scan at 0.42) -->
     <link name="lidar_post_fl">
-        <visual><geometry><box size="0.015 0.015 0.25"/></geometry><material name="black"/></visual>
-        <collision><geometry><box size="0.015 0.015 0.25"/></geometry></collision>
+        <visual><geometry><box size="0.015 0.015 0.33"/></geometry><material name="black"/></visual>
+        <collision><geometry><box size="0.015 0.015 0.33"/></geometry></collision>
         <inertial><mass value="0.15"/><origin xyz="0 0 0"/>
             <inertia ixx="0.001" ixy="0" ixz="0" iyy="0.001" iyz="0" izz="0.00005"/></inertial>
@@ -174,9 +174,9 @@
     <joint name="lidar_post_fl_joint" type="fixed">
         <parent link="base_link"/><child link="lidar_post_fl"/>
-        <origin xyz="0.20 0.07 0.265"/>
+        <origin xyz="0.20 0.07 0.225"/>
     </joint>
      <link name="lidar_post_fr">
-        <visual><geometry><box size="0.015 0.015 0.25"/></geometry><material name="black"/></visual>
-        <collision><geometry><box size="0.015 0.015 0.25"/></geometry></collision>
+        <visual><geometry><box size="0.015 0.015 0.33"/></geometry><material name="black"/></visual>
+        <collision><geometry><box size="0.015 0.015 0.33"/></geometry></collision>
         <inertial><mass value="0.15"/><origin xyz="0 0 0"/>
             <inertia ixx="0.001" ixy="0" ixz="0" iyy="0.001" iyz="0" izz="0.00005"/></inertial>
@@ -184,9 +184,9 @@
     <joint name="lidar_post_fr_joint" type="fixed">
         <parent link="base_link"/><child link="lidar_post_fr"/>
-        <origin xyz="0.20 -0.07 0.265"/>
+        <origin xyz="0.20 -0.07 0.225"/>
     </joint>
     <link name="lidar_post_rl">
-        <visual><geometry><box size="0.015 0.015 0.25"/></geometry><material name="black"/></visual>
-        <collision><geometry><box size="0.015 0.015 0.25"/></geometry></collision>
+        <visual><geometry><box size="0.015 0.015 0.33"/></geometry><material name="black"/></visual>
+        <collision><geometry><box size="0.015 0.015 0.33"/></geometry></collision>
         <inertial><mass value="0.15"/><origin xyz="0 0 0"/>
             <inertia ixx="0.001" ixy="0" ixz="0" iyy="0.001" iyz="0" izz="0.00005"/></inertial>
@@ -194,9 +194,9 @@
     <joint name="lidar_post_rl_joint" type="fixed">
         <parent link="base_link"/><child link="lidar_post_rl"/>
-        <origin xyz="0.08 0.07 0.265"/>
+        <origin xyz="-0.17 0.07 0.225"/>
     </joint>
     <link name="lidar_post_rr">
-        <visual><geometry><box size="0.015 0.015 0.25"/></geometry><material name="black"/></visual>
-        <collision><geometry><box size="0.015 0.015 0.25"/></geometry></collision>
+        <visual><geometry><box size="0.015 0.015 0.33"/></geometry><material name="black"/></visual>
+        <collision><geometry><box size="0.015 0.015 0.33"/></geometry></collision>
         <inertial><mass value="0.15"/><origin xyz="0 0 0"/>
             <inertia ixx="0.001" ixy="0" ixz="0" iyy="0.001" iyz="0" izz="0.00005"/></inertial>
@@ -204,5 +204,5 @@
     <joint name="lidar_post_rr_joint" type="fixed">
         <parent link="base_link"/><child link="lidar_post_rr"/>
-        <origin xyz="0.08 -0.07 0.265"/>
+        <origin xyz="-0.17 -0.07 0.225"/>
     </joint>
     <!-- Top plate tying all 4 posts together -->
