Commit message: Add URDF components for LiDAR and camera, and update chassis parameters

File: src/campus_robot/urdf/chassis.xacro (robot description, xacro)
@@ -1,11 +1,10 @@
 <?xml version="1.0"?>
 <robot xmlns:xacro="http://www.ros.org/wiki/xacro">
-    <!-- ===================================================== -->
-    <!-- Base Chassis                                           -->
-    <!-- ===================================================== -->
+    <!-- ============================= -->
+    <!-- Base Chassis                  -->
+    <!-- ============================= -->
     <link name="base_link">
-        <!-- Visual -->
         <visual>
-            <origin xyz="0 0 0.06" rpy="0 0 0"/>
+            <origin xyz="0 0 0.06"/>
             <geometry>
                 <box size="0.45 0.35 0.12"/>
@@ -13,54 +12,54 @@
             <material name="blue"/>
         </visual>
-        <!-- Collision -->
         <collision>
-            <origin xyz="0 0 0.06" rpy="0 0 0"/>
+            <origin xyz="0 0 0.06"/>
             <geometry>
                 <box size="0.45 0.35 0.12"/>
             </geometry>
         </collision>
-        <!-- Inertia -->
         <inertial>
-            <origin xyz="0 0 0.06" rpy="0 0 0"/>
-            <mass value="8.0"/>
+            <origin xyz="0 0 0.06"/>
+            <mass value="8"/>
             <inertia
-                ixx="0.120"
-                ixy="0.0"
-                ixz="0.0"
-                iyy="0.180"
-                iyz="0.0"
-                izz="0.250"/>
+                ixx="0.12"
+                ixy="0"
+                ixz="0"
+                iyy="0.18"
+                iyz="0"
+                izz="0.25"/>
         </inertial>
     </link>
-    <!-- ===================================================== -->
-    <!-- Parcel Box                                             -->
-    <!-- ===================================================== -->
+    <!-- ============================= -->
+    <!-- Parcel Box                    -->
+    <!-- ============================= -->
     <link name="parcel_box">
         <visual>
-            <origin xyz="0 0 0.17" rpy="0 0 0"/>
+            <origin xyz="0 0 0.22"/>
             <geometry>
-                <box size="0.25 0.20 0.10"/>
+                <box size="0.30 0.25 0.12"/>
             </geometry>
             <material name="grey"/>
         </visual>
         <collision>
-            <origin xyz="0 0 0.17" rpy="0 0 0"/>
+            <origin xyz="0 0 0.22"/>
             <geometry>
-                <box size="0.25 0.20 0.10"/>
+                <box size="0.30 0.25 0.12"/>
             </geometry>
         </collision>
         <inertial>
-            <origin xyz="0 0 0.17" rpy="0 0 0"/>
-            <mass value="1.0"/>
+            <origin xyz="0 0 0.22"/>
+            <mass value="1.5"/>
             <inertia
-                ixx="0.01"
+                ixx="0.02"
                 ixy="0"
                 ixz="0"
-                iyy="0.01"
+                iyy="0.02"
                 iyz="0"
-                izz="0.01"/>
+                izz="0.02"/>
         </inertial>
     </link>
-    <joint name="parcel_box_joint" type="fixed">
+    <joint
+        name="parcel_box_joint"
+        type="fixed">
         <parent link="base_link"/>
         <child link="parcel_box"/>

File: src/campus_robot/urdf/sensors.xacro (robot description, xacro)
@@ -1,11 +1,37 @@
 <?xml version="1.0"?>
 <robot xmlns:xacro="http://www.ros.org/wiki/xacro">
-    <!-- ===================================================== -->
-    <!-- LiDAR                                                 -->
-    <!-- ===================================================== -->
+    <!-- ===================================== -->
+    <!-- LiDAR Mast                            -->
+    <!-- ===================================== -->
+    <link name="lidar_mount">
+        <visual>
+            <geometry>
+                <cylinder radius="0.01"
+                          length="0.16"/>
+            </geometry>
+            <material name="black"/>
+        </visual>
+        <collision>
+            <geometry>
+                <cylinder radius="0.01"
+                          length="0.16"/>
+            </geometry>
+        </collision>
+    </link>
+    <joint
+        name="lidar_mount_joint"
+        type="fixed">
+        <parent link="base_link"/>
+        <child link="lidar_mount"/>
+        <origin xyz="0 0 0.20"/>
+    </joint>
+    <!-- ===================================== -->
+    <!-- LiDAR                                 -->
+    <!-- ===================================== -->
     <link name="lidar_link">
         <visual>
             <geometry>
-                <cylinder radius="0.04" length="0.05"/>
+                <cylinder radius="0.045"
+                          length="0.05"/>
             </geometry>
             <material name="dark_grey"/>
@@ -13,32 +39,24 @@
         <collision>
             <geometry>
-                <cylinder radius="0.04" length="0.05"/>
+                <cylinder radius="0.045"
+                          length="0.05"/>
             </geometry>
         </collision>
-        <inertial>
-            <mass value="0.20"/>
-            <origin xyz="0 0 0"/>
-            <inertia
-                ixx="0.0002"
-                ixy="0"
-                ixz="0"
-                iyy="0.0002"
-                iyz="0"
-                izz="0.0002"/>
-        </inertial>
     </link>
-    <joint name="lidar_joint" type="fixed">
-        <parent link="base_link"/>
+    <joint
+        name="lidar_joint"
+        type="fixed">
+        <parent link="lidar_mount"/>
         <child link="lidar_link"/>
-        <!-- Top center of chassis -->
-        <origin xyz="0.10 0 0.17"/>
+        <origin xyz="0 0 0.105"/>
     </joint>
-    <!-- ===================================================== -->
-    <!-- Camera                                                -->
-    <!-- ===================================================== -->
-    <link name="camera_link">
+    <!-- ===================================== -->
+    <!-- Camera Mount                          -->
+    <!-- ===================================== -->
+    <link name="camera_mount">
         <visual>
             <geometry>
-                <box size="0.04 0.04 0.04"/>
+                <cylinder radius="0.008"
+                          length="0.09"/>
             </geometry>
             <material name="black"/>
@@ -46,30 +64,44 @@
         <collision>
             <geometry>
-                <box size="0.04 0.04 0.04"/>
+                <cylinder radius="0.008"
+                          length="0.09"/>
             </geometry>
         </collision>
-        <inertial>
-            <mass value="0.15"/>
-            <origin xyz="0 0 0"/>
-            <inertia
-                ixx="0.0001"
-                ixy="0"
-                ixz="0"
-                iyy="0.0001"
-                iyz="0"
-                izz="0.0001"/>
-        </inertial>
     </link>
-    <joint name="camera_joint" type="fixed">
+    <joint
+        name="camera_mount_joint"
+        type="fixed">
         <parent link="base_link"/>
+        <child link="camera_mount"/>
+        <origin xyz="0.18 0 0.18"/>
+    </joint>
+    <!-- ===================================== -->
+    <!-- RGB Camera                            -->
+    <!-- ===================================== -->
+    <link name="camera_link">
+        <visual>
+            <geometry>
+                <box size="0.05 0.04 0.04"/>
+            </geometry>
+            <material name="black"/>
+        </visual>
+        <collision>
+            <geometry>
+                <box size="0.05 0.04 0.04"/>
+            </geometry>
+        </collision>
+    </link>
+    <joint
+        name="camera_joint"
+        type="fixed">
+        <parent link="camera_mount"/>
         <child link="camera_link"/>
-        <!-- Slightly forward and above the LiDAR -->
-        <origin xyz="0.18 0 0.17"/>
+        <origin xyz="0 0 0.065"
+                rpy="0.30 0 0"/>
     </joint>
-    <!-- ===================================================== -->
-    <!-- IMU                                                   -->
-    <!-- ===================================================== -->
+    <!-- ===================================== -->
+    <!-- IMU                                   -->
+    <!-- ===================================== -->
     <link name="imu_link">
-        <!-- IMU is tiny; keep it invisible -->
         <visual>
             <geometry>
@@ -78,26 +110,11 @@
             <material name="orange"/>
         </visual>
-        <collision>
-            <geometry>
-                <box size="0.02 0.02 0.01"/>
-            </geometry>
-        </collision>
-        <inertial>
-            <mass value="0.05"/>
-            <origin xyz="0 0 0"/>
-            <inertia
-                ixx="0.00001"
-                ixy="0"
-                ixz="0"
-                iyy="0.00001"
-                iyz="0"
-                izz="0.00001"/>
-        </inertial>
     </link>
-    <joint name="imu_joint" type="fixed">
+    <joint
+        name="imu_joint"
+        type="fixed">
         <parent link="base_link"/>
         <child link="imu_link"/>
-        <!-- Near the center of gravity -->
-        <origin xyz="0 0 0.10"/>
+        <origin xyz="0 0 0.09"/>
     </joint>
 </robot>

Commit message: Refactor URDF files for sensor tower and adjust dimensions for LiDAR and camera components

File: src/campus_robot/urdf/chassis.xacro (robot description, xacro)
@@ -35,5 +35,5 @@
     <link name="parcel_box">
         <visual>
-            <origin xyz="0 0 0.22"/>
+            <origin xyz="0 0 0.18"/>
             <geometry>
                 <box size="0.30 0.25 0.12"/>
@@ -42,5 +42,5 @@
         </visual>
         <collision>
-            <origin xyz="0 0 0.22"/>
+            <origin xyz="0 0 0.18"/>
             <geometry>
                 <box size="0.30 0.25 0.12"/>
@@ -48,5 +48,5 @@
         </collision>
         <inertial>
-            <origin xyz="0 0 0.22"/>
+            <origin xyz="0 0 0.18"/>
             <mass value="1.5"/>
             <inertia

File: src/campus_robot/urdf/sensors.xacro (robot description, xacro)
@@ -1,12 +1,11 @@
 <?xml version="1.0"?>
 <robot xmlns:xacro="http://www.ros.org/wiki/xacro">
-    <!-- ===================================== -->
-    <!-- LiDAR Mast                            -->
-    <!-- ===================================== -->
-    <link name="lidar_mount">
+    <!-- ================================ -->
+    <!-- Sensor Tower                     -->
+    <!-- ================================ -->
+    <link name="sensor_tower">
         <visual>
             <geometry>
-                <cylinder radius="0.01"
-                          length="0.16"/>
+                <box size="0.05 0.05 0.14"/>
             </geometry>
             <material name="black"/>
@@ -14,15 +13,25 @@
         <collision>
             <geometry>
-                <cylinder radius="0.01"
-                          length="0.16"/>
+                <box size="0.05 0.05 0.14"/>
             </geometry>
         </collision>
+        <inertial>
+            <mass value="0.5"/>
+            <origin xyz="0 0 0"/>
+            <inertia
+                ixx="0.001"
+                ixy="0"
+                ixz="0"
+                iyy="0.001"
+                iyz="0"
+                izz="0.001"/>
+        </inertial>
     </link>
     <joint
-        name="lidar_mount_joint"
+        name="sensor_tower_joint"
         type="fixed">
         <parent link="base_link"/>
-        <child link="lidar_mount"/>
-        <origin xyz="0 0 0.20"/>
+        <child link="sensor_tower"/>
+        <origin xyz="0.14 0 0.19"/>
     </joint>
     <!-- ===================================== -->
@@ -47,7 +56,7 @@
         name="lidar_joint"
         type="fixed">
-        <parent link="lidar_mount"/>
+        <parent link="sensor_tower"/>
         <child link="lidar_link"/>
-        <origin xyz="0 0 0.105"/>
+        <origin xyz="0 0 0.095"/>
     </joint>
     <!-- ===================================== -->
@@ -57,13 +66,11 @@
         <visual>
             <geometry>
-                <cylinder radius="0.008"
-                          length="0.09"/>
+                <box size="0.03 0.03 0.05"/>
             </geometry>
-            <material name="black"/>
+            <material name="dark_grey"/>
         </visual>
         <collision>
             <geometry>
-                <cylinder radius="0.008"
-                          length="0.09"/>
+                <box size="0.03 0.03 0.05"/>
             </geometry>
         </collision>
@@ -72,7 +79,7 @@
         name="camera_mount_joint"
         type="fixed">
-        <parent link="base_link"/>
+        <parent link="sensor_tower"/>
         <child link="camera_mount"/>
-        <origin xyz="0.18 0 0.18"/>
+        <origin xyz="0.05 0 0.02"/>
     </joint>
     <!-- ===================================== -->
@@ -97,6 +104,6 @@
         <parent link="camera_mount"/>
         <child link="camera_link"/>
-        <origin xyz="0 0 0.065"
-                rpy="0.30 0 0"/>
+        <origin xyz="0.04 0 0"
+                rpy="0 -0.25 0"/>
     </joint>
     <!-- ===================================== -->

Commit message: Refactor gazebo launch file to use TimerAction for robot spawning; adjust spawn position and update chassis URDF parameters for improved stability and performance

File: src/campus_robot/urdf/chassis.xacro (robot description, xacro)
@@ -13,17 +13,17 @@
         </visual>
         <collision>
-            <origin xyz="0 0 0.06"/>
+            <origin xyz="0 0 0.075"/>
             <geometry>
-                <box size="0.45 0.35 0.12"/>
+                <box size="0.45 0.35 0.10"/>
             </geometry>
         </collision>
         <inertial>
-            <origin xyz="0 0 0.06"/>
-            <mass value="8"/>
+            <origin xyz="0 0 0.075"/>
+            <mass value="15"/>
             <inertia
                 ixx="0.12"
                 ixy="0"
                 ixz="0"
-                iyy="0.18"
+                iyy="0.40"
                 iyz="0"
                 izz="0.25"/>

File: src/campus_robot/urdf/gazebo_plugins.xacro (robot description, xacro)
@@ -10,12 +10,21 @@
     </gazebo>
     <gazebo reference="left_wheel">
-        <material>Gazebo/Black</material>
-        <mu1>5.0</mu1>
-        <mu2>5.0</mu2>
+        <mu1>20</mu1>
+        <mu2>20</mu2>
+        <kp>1000000</kp>
+        <kd>100</kd>
     </gazebo>
     <gazebo reference="right_wheel">
-        <material>Gazebo/Black</material>
-        <mu1>5.0</mu1>
-        <mu2>5.0</mu2>
+        <mu1>20</mu1>
+        <mu2>20</mu2>
+        <kp>1000000</kp>
+        <kd>100</kd>
+    </gazebo>
+    <gazebo reference="caster_wheel">
+        <mu1>0.05</mu1>
+        <mu2>0.05</mu2>
+        <kp>1000000</kp>
+        <kd>100</kd>
+        <material>Gazebo/Grey</material>
     </gazebo>
     <!-- ========================================================= -->
@@ -36,6 +45,6 @@
             <wheel_diameter>0.14</wheel_diameter>
             <!-- Motion limits -->
-            <max_wheel_torque>30</max_wheel_torque>
-            <max_wheel_acceleration>8.0</max_wheel_acceleration>
+            <max_wheel_torque>10</max_wheel_torque>
+            <max_wheel_acceleration>1</max_wheel_acceleration>
             <!-- Topics -->
             <command_topic>cmd_vel</command_topic>
@@ -48,4 +57,5 @@
             <publish_odom_tf>true</publish_odom_tf>
             <publish_wheel_tf>false</publish_wheel_tf>
+            <publish_wheel_joint_state>true</publish_wheel_joint_state>
             <!-- Legacy mode -->
             <legacy_mode>false</legacy_mode>

File: src/campus_robot/urdf/wheels.xacro (robot description, xacro)
@@ -40,5 +40,5 @@
         <parent link="base_link"/>
         <child link="left_wheel"/>
-        <origin xyz="0 0.195 0.07"/>
+        <origin xyz="0 0.195 0.075"/>
         <axis xyz="0 1 0"/>
     </joint>
@@ -77,5 +77,5 @@
         <parent link="base_link"/>
         <child link="right_wheel"/>
-        <origin xyz="0 -0.195 0.07"/>
+        <origin xyz="0 -0.195 0.075"/>
         <axis xyz="0 1 0"/>
     </joint>
@@ -111,5 +111,5 @@
         <parent link="base_link"/>
         <child link="caster_wheel"/>
-        <origin xyz="-0.17 0 0.03"/>
+        <origin xyz="-0.15 0 0.03"/>
     </joint>
 </robot>

Commit message: Add joint state publisher and adjust robot dimensions; implement rear caster wheels with updated parameters

File: src/campus_robot/urdf/chassis.xacro (robot description, xacro)
@@ -6,5 +6,5 @@
     <link name="base_link">
         <visual>
-            <origin xyz="0 0 0.06"/>
+            <origin xyz="0 0 0.06" rpy="0 0 0"/>
             <geometry>
                 <box size="0.45 0.35 0.12"/>
@@ -13,19 +13,19 @@
         </visual>
         <collision>
-            <origin xyz="0 0 0.075"/>
+            <origin xyz="0 0 0.06" rpy="0 0 0"/>
             <geometry>
-                <box size="0.45 0.35 0.10"/>
+                <box size="0.45 0.25 0.10"/>
             </geometry>
         </collision>
         <inertial>
-            <origin xyz="0 0 0.075"/>
+            <origin xyz="0 0 0.06"/>
             <mass value="15"/>
             <inertia
-                ixx="0.12"
+                ixx="0.25"
                 ixy="0"
                 ixz="0"
                 iyy="0.40"
                 iyz="0"
-                izz="0.25"/>
+                izz="0.50"/>
         </inertial>
     </link>
@@ -66,3 +66,38 @@
         <origin xyz="0 0 0.12"/>
     </joint>
+    <!-- ============================= -->
+    <!-- Rear Support Rod              -->
+    <!-- ============================= -->
+    <link name="rear_support_rod">
+        <visual>
+            <origin xyz="0 0 0" rpy="0 0 0"/>
+            <geometry>
+                <box size="0.05 0.05 0.14"/>   <!-- same dimensions as sensor_tower -->
+            </geometry>
+            <material name="black"/>
+        </visual>
+        <collision>
+            <origin xyz="0 0 0" rpy="0 0 0"/>
+            <geometry>
+                <box size="0.05 0.05 0.14"/>
+            </geometry>
+        </collision>
+        <inertial>
+            <mass value="0.5"/>
+            <origin xyz="0 0 0"/>
+            <inertia
+                ixx="0.001"
+                ixy="0"
+                ixz="0"
+                iyy="0.001"
+                iyz="0"
+                izz="0.001"/>
+        </inertial>
+    </link>
+    <joint name="rear_support_rod_joint" type="fixed">
+        <parent link="base_link"/>
+        <child link="rear_support_rod"/>
+        <!-- sensor_tower is at x=+0.14, so mirror it to rear at x=-0.14 -->
+        <origin xyz="-0.14 0 0.19"/>
+    </joint>
 </robot>

File: src/campus_robot/urdf/gazebo_plugins.xacro (robot description, xacro)
@@ -21,7 +21,14 @@
         <kd>100</kd>
     </gazebo>
-    <gazebo reference="caster_wheel">
-        <mu1>0.05</mu1>
-        <mu2>0.05</mu2>
+    <gazebo reference="caster_wheel_left">
+        <mu1>0.01</mu1>
+        <mu2>0.01</mu2>
+        <kp>1000000</kp>
+        <kd>100</kd>
+        <material>Gazebo/Grey</material>
+    </gazebo>
+    <gazebo reference="caster_wheel_right">
+        <mu1>0.01</mu1>
+        <mu2>0.01</mu2>
         <kp>1000000</kp>
         <kd>100</kd>
@@ -57,5 +64,5 @@
             <publish_odom_tf>true</publish_odom_tf>
             <publish_wheel_tf>false</publish_wheel_tf>
-            <publish_wheel_joint_state>true</publish_wheel_joint_state>
+            <publish_wheel_joint_state>false</publish_wheel_joint_state>
             <!-- Legacy mode -->
             <legacy_mode>false</legacy_mode>

File: src/campus_robot/urdf/wheels.xacro (robot description, xacro)
@@ -81,10 +81,10 @@
     </joint>
     <!-- ============================= -->
-    <!-- Rear Caster Wheel             -->
+    <!-- Rear Caster Left              -->
     <!-- ============================= -->
-    <link name="caster_wheel">
+    <link name="caster_wheel_left">
         <visual>
             <geometry>
-                <sphere radius="0.03"/>
+                <sphere radius="0.04"/>   <!-- bigger radius — more stable -->
             </geometry>
             <material name="grey"/>
@@ -92,24 +92,55 @@
         <collision>
             <geometry>
-                <sphere radius="0.03"/>
+                <sphere radius="0.04"/>
             </geometry>
         </collision>
         <inertial>
-            <mass value="0.2"/>
+            <mass value="0.3"/>
             <origin xyz="0 0 0"/>
             <inertia
-                ixx="0.0002"
+                ixx="0.0003"
                 ixy="0"
                 ixz="0"
-                iyy="0.0002"
+                iyy="0.0003"
                 iyz="0"
-                izz="0.0002"/>
+                izz="0.0003"/>
         </inertial>
     </link>
-    <joint name="caster_joint"
-           type="fixed">
+    <joint name="caster_left_joint" type="fixed">
         <parent link="base_link"/>
-        <child link="caster_wheel"/>
-        <origin xyz="-0.15 0 0.03"/>
+        <child link="caster_wheel_left"/>
+        <origin xyz="-0.17 0.10 0.05"/>  <!-- rear, spread left -->
+    </joint>
+    <!-- ============================= -->
+    <!-- Rear Caster Right             -->
+    <!-- ============================= -->
+    <link name="caster_wheel_right">
+        <visual>
+            <geometry>
+                <sphere radius="0.04"/>
+            </geometry>
+            <material name="grey"/>
+        </visual>
+        <collision>
+            <geometry>
+                <sphere radius="0.04"/>
+            </geometry>
+        </collision>
+        <inertial>
+            <mass value="0.3"/>
+            <origin xyz="0 0 0"/>
+            <inertia
+                ixx="0.0003"
+                ixy="0"
+                ixz="0"
+                iyy="0.0003"
+                iyz="0"
+                izz="0.0003"/>
+        </inertial>
+    </link>
+    <joint name="caster_right_joint" type="fixed">
+        <parent link="base_link"/>
+        <child link="caster_wheel_right"/>
+        <origin xyz="-0.17 -0.10 0.05"/>  <!-- rear, spread right -->
     </joint>
 </robot>

Commit message: Adjust chassis collision height and update road model dimensions for improved simulation accuracy

File: src/campus_robot/urdf/chassis.xacro (robot description, xacro)
@@ -13,5 +13,5 @@
         </visual>
         <collision>
-            <origin xyz="0 0 0.06" rpy="0 0 0"/>
+            <origin xyz="0 0 0.07" rpy="0 0 0"/>
             <geometry>
                 <box size="0.45 0.25 0.10"/>
