Commit message: Add SLAM parameters, update map configurations, and refine URDF for improved simulation accuracy

File: src/campus_robot/urdf/chassis.xacro (robot description, xacro)
@@ -25,5 +25,5 @@
                 ixy="0"
                 ixz="0"
-                iyy="0.40"
+                iyy="1.20"
                 iyz="0"
                 izz="0.50"/>

File: src/campus_robot/urdf/gazebo_plugins.xacro (robot description, xacro)
@@ -29,4 +29,18 @@
     </gazebo>
     <gazebo reference="caster_wheel_right">
+        <mu1>0.01</mu1>
+        <mu2>0.01</mu2>
+        <kp>1000000</kp>
+        <kd>100</kd>
+        <material>Gazebo/Grey</material>
+    </gazebo>
+    <gazebo reference="caster_front_left">
+        <mu1>0.01</mu1>
+        <mu2>0.01</mu2>
+        <kp>1000000</kp>
+        <kd>100</kd>
+        <material>Gazebo/Grey</material>
+    </gazebo>
+    <gazebo reference="caster_front_right">
         <mu1>0.01</mu1>
         <mu2>0.01</mu2>
@@ -75,8 +89,11 @@
         <sensor name="imu_sensor" type="imu">
             <always_on>true</always_on>
+            <!-- 100 Hz is ideal -->
             <update_rate>100</update_rate>
+            <!-- Optional -->
             <visualize>false</visualize>
-            <plugin name="imu_plugin"
-                    filename="libgazebo_ros_imu_sensor.so">
+            <plugin
+                name="imu_plugin"
+                filename="libgazebo_ros_imu_sensor.so">
                 <ros>
                     <remapping>~/out:=imu</remapping>
@@ -98,5 +115,5 @@
                 <scan>
                     <horizontal>
-                        <samples>720</samples>
+                        <samples>1080</samples>
                         <resolution>1</resolution>
                         <min_angle>-3.14159</min_angle>
@@ -105,8 +122,13 @@
                 </scan>
                 <range>
-                    <min>0.10</min>
+                    <min>0.25</min>
                     <max>20.0</max>
-                    <resolution>0.01</resolution>
+                    <resolution>0.005</resolution>
                 </range>
+                <noise>
+                    <type>gaussian</type>
+                    <mean>0.0</mean>
+                    <stddev>0.01</stddev>
+                </noise>
             </ray>
             <plugin

File: src/campus_robot/urdf/sensors.xacro (robot description, xacro)
@@ -103,5 +103,5 @@
         <parent link="lidar_base_link"/>
         <child  link="lidar_link"/>
-        <origin xyz="0.0 0.0 0.03" rpy="0 0 0"/>
+        <origin xyz="0.0 0.0 0.03" rpy="0 -0.035 0"/>
     </joint>
     <!-- ===================================== -->
@@ -164,3 +164,38 @@
         <origin xyz="0 0 0.09"/>
     </joint>
+    <!-- 4-Corner LiDAR Frame: FL, FR, RL, RR posts -->
+    <!-- bottom z=0.14 (2mm above chassis top), top z=0.39 (below LiDAR scan at 0.42) -->
+    <link name="lidar_post_fl">
+        <visual><geometry><box size="0.015 0.015 0.25"/></geometry><material name="black"/></visual>
+        <collision><geometry><box size="0.015 0.015 0.25"/></geometry></collision>
+        <inertial><mass value="0.15"/><origin xyz="0 0 0"/>
+            <inertia ixx="0.001" ixy="0" ixz="0" iyy="0.001" iyz="0" izz="0.00005"/></inertial>
+    </link>
+    <joint name="lidar_post_fl_joint" type="fixed">
+        <parent link="base_link"/><child link="lidar_post_fl"/>
+        <origin xyz="0.20 0.07 0.265"/>
+    </joint>
+    <link name="lidar_post_fr">  ... same geometry ...  </link>
+    <joint name="lidar_post_fr_joint" type="fixed">
+        <origin xyz="0.20 -0.07 0.265"/>
+    </joint>
+    <link name="lidar_post_rl">  ... same geometry ...  </link>
+    <joint name="lidar_post_rl_joint" type="fixed">
+        <origin xyz="0.08 0.07 0.265"/>
+    </joint>
+    <link name="lidar_post_rr">  ... same geometry ...  </link>
+    <joint name="lidar_post_rr_joint" type="fixed">
+        <origin xyz="0.08 -0.07 0.265"/>
+    </joint>
+    <!-- Top plate tying all 4 posts together -->
+    <link name="lidar_top_plate">
+        <visual><geometry><box size="0.16 0.16 0.01"/></geometry><material name="black"/></visual>
+        <collision><geometry><box size="0.16 0.16 0.01"/></geometry></collision>
+        <inertial><mass value="0.1"/><origin xyz="0 0 0"/>
+            <inertia ixx="0.0001" ixy="0" ixz="0" iyy="0.0001" iyz="0" izz="0.0002"/></inertial>
+    </link>
+    <joint name="lidar_top_plate_joint" type="fixed">
+        <parent link="base_link"/><child link="lidar_top_plate"/>
+        <origin xyz="0.14 0.0 0.395"/>
+    </joint>
 </robot>

File: src/campus_robot/urdf/wheels.xacro (robot description, xacro)
@@ -110,5 +110,5 @@
         <parent link="base_link"/>
         <child link="caster_wheel_left"/>
-        <origin xyz="-0.17 0.10 0.06"/>  <!-- rear, spread left -->
+        <origin xyz="-0.20 0.10 0.06"/>  <!-- rear, spread left -->
     </joint>
     <!-- ============================= -->
@@ -142,5 +142,47 @@
         <parent link="base_link"/>
         <child link="caster_wheel_right"/>
-        <origin xyz="-0.17 -0.10 0.06"/>  <!-- rear, spread right -->
+        <origin xyz="-0.20 -0.10 0.06"/>  <!-- rear, spread right -->
+    </joint>
+    <!-- Front Caster Left -->
+    <link name="caster_front_left">
+        <visual>
+            <geometry><sphere radius="0.05"/></geometry>
+            <material name="grey"/>
+        </visual>
+        <collision>
+            <geometry><sphere radius="0.05"/></geometry>
+        </collision>
+        <inertial>
+            <mass value="0.3"/>
+            <origin xyz="0 0 0"/>
+            <inertia ixx="0.0003" ixy="0" ixz="0"
+                    iyy="0.0003" iyz="0" izz="0.0003"/>
+        </inertial>
+    </link>
+    <joint name="caster_front_left_joint" type="fixed">
+        <parent link="base_link"/>
+        <child link="caster_front_left"/>
+        <origin xyz="0.17 0.10 0.06"/>
+    </joint>
+    <!-- Front Caster Right -->
+    <link name="caster_front_right">
+        <visual>
+            <geometry><sphere radius="0.05"/></geometry>
+            <material name="grey"/>
+        </visual>
+        <collision>
+            <geometry><sphere radius="0.05"/></geometry>
+        </collision>
+        <inertial>
+            <mass value="0.3"/>
+            <origin xyz="0 0 0"/>
+            <inertia ixx="0.0003" ixy="0" ixz="0"
+                    iyy="0.0003" iyz="0" izz="0.0003"/>
+        </inertial>
+    </link>
+    <joint name="caster_front_right_joint" type="fixed">
+        <parent link="base_link"/>
+        <child link="caster_front_right"/>
+        <origin xyz="0.17 -0.10 0.06"/>
     </joint>
 </robot>

Commit message: Add battery pack to chassis URDF, adjust wheel joint origins, and modify max wheel acceleration for improved stability and performance

File: src/campus_robot/urdf/chassis.xacro (robot description, xacro)
@@ -101,3 +101,41 @@
         <origin xyz="-0.14 0 0.19"/>
     </joint>
+    <!-- ============================= -->
+    <!-- Battery Pack                  -->
+    <!-- Front section, low mount      -->
+    <!-- Shifts CoM forward to resist  -->
+    <!-- backward tipping on accel     -->
+    <!-- ============================= -->
+    <link name="battery_pack">
+        <visual>
+            <origin xyz="0 0 0"/>
+            <geometry>
+                <box size="0.18 0.28 0.05"/>
+            </geometry>
+            <material name="black"/>
+        </visual>
+        <collision>
+            <origin xyz="0 0 0"/>
+            <geometry>
+                <box size="0.18 0.28 0.05"/>
+            </geometry>
+        </collision>
+        <inertial>
+            <mass value="3.0"/>
+            <origin xyz="0 0 0"/>
+            <inertia
+                ixx="0.010"
+                ixy="0"
+                ixz="0"
+                iyy="0.008"
+                iyz="0"
+                izz="0.016"/>
+        </inertial>
+    </link>
+    <joint name="battery_joint" type="fixed">
+        <parent link="base_link"/>
+        <child link="battery_pack"/>
+        <!-- front section of chassis, sitting on floor -->
+        <origin xyz="0.10 0 0.045"/>
+    </joint>
 </robot>

File: src/campus_robot/urdf/gazebo_plugins.xacro (robot description, xacro)
@@ -67,5 +67,5 @@
             <!-- Motion limits -->
             <max_wheel_torque>20</max_wheel_torque>
-            <max_wheel_acceleration>1</max_wheel_acceleration>
+            <max_wheel_acceleration>0.4</max_wheel_acceleration>
             <!-- Topics -->
             <command_topic>cmd_vel</command_topic>

File: src/campus_robot/urdf/wheels.xacro (robot description, xacro)
@@ -163,5 +163,5 @@
         <parent link="base_link"/>
         <child link="caster_front_left"/>
-        <origin xyz="0.17 0.10 0.06"/>
+        <origin xyz="0.22 0.10 0.06"/>
     </joint>
     <!-- Front Caster Right -->
@@ -184,5 +184,5 @@
         <parent link="base_link"/>
         <child link="caster_front_right"/>
-        <origin xyz="0.17 -0.10 0.06"/>
+        <origin xyz="0.22 -0.10 0.06"/>
     </joint>
 </robot>
