Commit message: Update navigation parameters and camera frame configurations for improved obstacle avoidance and vision processing. Adjusted BaseObstacle scale and costmap inflation parameters for better navigation performance. Modified camera frame name to ensure correct depth data alignment in the costmap.

File: src/campus_robot/urdf/gazebo_plugins.xacro (robot description, xacro)
@@ -176,9 +176,15 @@
                 name="camera_plugin"
                 filename="libgazebo_ros_camera.so">
-                <!-- Fixed name/frame so ROS topics are deterministic:
+                <!-- Fixed name so ROS topics are deterministic:
                      /camera_link/image_raw, /camera_link/depth/image_raw,
                      /camera_link/depth/camera_info, /camera_link/points -->
                 <camera_name>camera_link</camera_name>
-                <frame_name>camera_link</frame_name>
+                <!-- The plugin generates depth/point-cloud data in OPTICAL
+                     convention (Z forward, X right, Y down), so the frame_id
+                     it stamps on messages must be the optical child frame
+                     (see sensors.xacro), not the physical camera_link
+                     (X-forward, Z-up). Using the wrong frame here silently
+                     misplaces every vision-based obstacle in the costmap. -->
+                <frame_name>camera_link_optical</frame_name>
                 <min_depth>0.1</min_depth>
                 <max_depth>10.0</max_depth>

File: src/campus_robot/urdf/sensors.xacro (robot description, xacro)
@@ -147,4 +147,25 @@
     </joint>
     <!-- ===================================== -->
+    <!-- Camera Optical Frame                  -->
+    <!-- REP-103 optical convention: Z forward -->
+    <!-- into the scene, X right, Y down. The  -->
+    <!-- Gazebo depth camera plugin computes   -->
+    <!-- depth/point-cloud data in THIS frame, -->
+    <!-- so gazebo_plugins.xacro must publish  -->
+    <!-- with frame_name=camera_link_optical   -->
+    <!-- (not the physical camera_link, whose  -->
+    <!-- axes are X-forward/Z-up) or vision    -->
+    <!-- obstacles land in the wrong place.    -->
+    <!-- ===================================== -->
+    <link name="camera_link_optical"/>
+    <joint
+        name="camera_optical_joint"
+        type="fixed">
+        <parent link="camera_link"/>
+        <child link="camera_link_optical"/>
+        <origin xyz="0 0 0"
+                rpy="-1.5708 0 -1.5708"/>
+    </joint>
+    <!-- ===================================== -->
     <!-- IMU                                   -->
     <!-- ===================================== -->
